File: devboard.kicad_sch (KiCad schematic)
At the start: 39 parts, among them J1 USB4110-GF-A, J2 USB_BOOT, P1 TC2030-CTX, U1 RP2040, U2 NCP1117-3.3_SOT223, U3 AT25SF128A-SHB-T, Y1 ECS-2033-120-BN

Commit message: Change board size
Parts:
- C1, C10, C11, C12, C13, C14, C2, C3, C4, C5, C6, C7, C8, C9: footprint Capacitor_SMD:C_0402_1005Metric -> 1A_Passives:C_0402_1005Metric_NoSilk
- R1, R2, R3, R4, R5, R6, R8: footprint Resistor_SMD:R_0402_1005Metric -> 1A_Passives:R_0402_1005Metric_WideSilk
Changed lines of the file:
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@@
       (effects (font (size 1.27 1.27)) (justify left))
     )
-    (property "Footprint" "Capacitor_SMD:C_0402_1005Metric" (at 182.88 33.02 0)
+    (property "Footprint" "1A_Passives:C_0402_1005Metric_NoSilk" (at 182.88 33.02 0)
       (effects (font (size 1.27 1.27)) hide)
     )
@@
       (effects (font (size 1.27 1.27)) (justify left))
     )
-    (property "Footprint" "Resistor_SMD:R_0402_1005Metric" (at 106.68 172.72 0)
+    (property "Footprint" "1A_Passives:R_0402_1005Metric_WideSilk" (at 106.68 172.72 0)
       (effects (font (size 1.27 1.27)) hide)
     )
@@
       (effects (font (size 1.27 1.27)) (justify left))
     )
-    (property "Footprint" "Capacitor_SMD:C_0402_1005Metric" (at 222.25 33.02 0)
+    (property "Footprint" "1A_Passives:C_0402_1005Metric_NoSilk" (at 222.25 33.02 0)
       (effects (font (size 1.27 1.27)) hide)
     )
@@
       (effects (font (size 1.27 1.27)) (justify right))
     )
-    (property "Footprint" "Resistor_SMD:R_0402_1005Metric" (at 24.13 177.8 0)
+    (property "Footprint" "1A_Passives:R_0402_1005Metric_WideSilk" (at 24.13 177.8 0)
       (effects (font (size 1.27 1.27)) hide)
     )
@@
       (effects (font (size 1.27 1.27)) (justify left))
     )
-    (property "Footprint" "Capacitor_SMD:C_0402_1005Metric" (at 252.73 33.02 0)
+    (property "Footprint" "1A_Passives:C_0402_1005Metric_NoSilk" (at 252.73 33.02 0)
       (effects (font (size 1.27 1.27)) hide)
     )
@@
       (effects (font (size 1.27 1.27)) (justify left))
     )
-    (property "Footprint" "Resistor_SMD:R_0402_1005Metric" (at 57.15 133.35 0)
+    (property "Footprint" "1A_Passives:R_0402_1005Metric_WideSilk" (at 57.15 133.35 0)
       (effects (font (size 1.27 1.27)) hide)
     )
@@
       (effects (font (size 1.27 1.27)) (justify left))
     )
-    (property "Footprint" "Resistor_SMD:R_0402_1005Metric" (at 26.67 177.8 0)
+    (property "Footprint" "1A_Passives:R_0402_1005Metric_WideSilk" (at 26.67 177.8 0)
       (effects (font (size 1.27 1.27)) hide)
     )
@@
       (effects (font (size 1.27 1.27)) (justify left))
     )
-    (property "Footprint" "Capacitor_SMD:C_0402_1005Metric" (at 224.79 52.07 0)
+    (property "Footprint" "1A_Passives:C_0402_1005Metric_NoSilk" (at 224.79 52.07 0)
       (effects (font (size 1.27 1.27)) hide)
     )
@@
       (effects (font (size 1.27 1.27)) (justify left))
     )
-    (property "Footprint" "Capacitor_SMD:C_0402_1005Metric" (at 232.41 33.02 0)
+    (property "Footprint" "1A_Passives:C_0402_1005Metric_NoSilk" (at 232.41 33.02 0)
       (effects (font (size 1.27 1.27)) hide)
     )
@@
       (effects (font (size 1.27 1.27)) (justify left))
     )
-    (property "Footprint" "Capacitor_SMD:C_0402_1005Metric" (at 193.04 33.02 0)
+    (property "Footprint" "1A_Passives:C_0402_1005Metric_NoSilk" (at 193.04 33.02 0)
       (effects (font (size 1.27 1.27)) hide)
     )
@@
       (effects (font (size 1.27 1.27)) (justify left))
     )
-    (property "Footprint" "Capacitor_SMD:C_0402_1005Metric" (at 273.05 33.02 0)
+    (property "Footprint" "1A_Passives:C_0402_1005Metric_NoSilk" (at 273.05 33.02 0)
       (effects (font (size 1.27 1.27)) hide)
     )
@@
       (effects (font (size 1.27 1.27)) (justify left))
     )
-    (property "Footprint" "Capacitor_SMD:C_0402_1005Metric" (at 262.89 33.02 0)
+    (property "Footprint" "1A_Passives:C_0402_1005Metric_NoSilk" (at 262.89 33.02 0)
       (effects (font (size 1.27 1.27)) hide)
     )
@@
       (effects (font (size 1.27 1.27)) (justify left))
     )
-    (property "Footprint" "Capacitor_SMD:C_0402_1005Metric" (at 77.47 135.89 0)
+    (property "Footprint" "1A_Passives:C_0402_1005Metric_NoSilk" (at 77.47 135.89 0)
       (effects (font (size 1.27 1.27)) hide)
     )
@@
       (effects (font (size 1.27 1.27)) (justify left))
     )
-    (property "Footprint" "Capacitor_SMD:C_0402_1005Metric" (at 242.57 33.02 0)
+    (property "Footprint" "1A_Passives:C_0402_1005Metric_NoSilk" (at 242.57 33.02 0)
       (effects (font (size 1.27 1.27)) hide)
     )
@@
       (effects (font (size 1.27 1.27)) (justify left))
     )
-    (property "Footprint" "Capacitor_SMD:C_0402_1005Metric" (at 157.48 168.91 0)
+    (property "Footprint" "1A_Passives:C_0402_1005Metric_NoSilk" (at 157.48 168.91 0)
       (effects (font (size 1.27 1.27)) hide)
     )
@@
       (effects (font (size 1.27 1.27)) (justify right))
     )
-    (property "Footprint" "Resistor_SMD:R_0402_1005Metric" (at 30.48 165.1 0)
+    (property "Footprint" "1A_Passives:R_0402_1005Metric_WideSilk" (at 30.48 165.1 0)
       (effects (font (size 1.27 1.27)) hide)
     )
@@
       (effects (font (size 1.27 1.27)) (justify left))
     )
-    (property "Footprint" "Capacitor_SMD:C_0402_1005Metric" (at 196.85 52.07 0)
+    (property "Footprint" "1A_Passives:C_0402_1005Metric_NoSilk" (at 196.85 52.07 0)
       (effects (font (size 1.27 1.27)) hide)
     )
@@
       (effects (font (size 1.27 1.27)) (justify left))
     )
-    (property "Footprint" "Capacitor_SMD:C_0402_1005Metric" (at 212.09 33.02 0)
+    (property "Footprint" "1A_Passives:C_0402_1005Metric_NoSilk" (at 212.09 33.02 0)
       (effects (font (size 1.27 1.27)) hide)
     )
@@
       (effects (font (size 1.27 1.27)) (justify right))
     )
-    (property "Footprint" "Resistor_SMD:R_0402_1005Metric" (at 25.4 165.1 0)
+    (property "Footprint" "1A_Passives:R_0402_1005Metric_WideSilk" (at 25.4 165.1 0)
       (effects (font (size 1.27 1.27)) hide)
     )
@@
       (effects (font (size 1.27 1.27)) (justify left))
     )
-    (property "Footprint" "Capacitor_SMD:C_0402_1005Metric" (at 101.6 135.89 0)
+    (property "Footprint" "1A_Passives:C_0402_1005Metric_NoSilk" (at 101.6 135.89 0)
       (effects (font (size 1.27 1.27)) hide)
     )
@@
       (effects (font (size 1.27 1.27)))
     )
-    (property "Footprint" "Resistor_SMD:R_0402_1005Metric" (at 99.06 177.8 0)
-      (effects (font (size 1.27 1.27)) hide)
-    )
+    (property "Footprint" "1A_Passives:R_0402_1005Metric_WideSilk" (at 99.06 177.8 0)
+      (effects (font (size 1.27 1.27)) hide)
+    )
