File: untitled.kicad_sch (KiCad schematic)
At the start: 168 parts, among them SW1 ESC, SW10 F9, SW11 F10, SW12 F11, SW13 F12, SW14 PRTSC, SW15 PAUSE, SW16 DEL, SW17 GRAVE, SW18 1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

Commit message: Change board size
Parts:
- SW1, SW10, SW11, SW12, SW13, SW14, SW15, SW16, SW17, SW18, SW19, SW2, SW20, SW21, SW22, SW23, SW24, SW25, SW26, SW27, SW28, SW29, SW3, SW31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: footprint Button_Switch_Keyboard:SW_Cherry_MX_1.00u_PCB -> 1A_Connectors:SW_Cherry_MX_1.00u_PCB
